Commit message: updated robot urdf file

File: robot_pybullet/robot.urdf (robot description, URDF)
Before this commit: robot three_dof_robot, 4 links, 3 joints
Links:
- link base: mass None -> 1.0
- link base_link: mass None -> 0.20
- link gripper: mass None -> 0.15
- link linker: mass None -> 0.15
Joints:
- removed joint joint1
- removed joint joint2
- removed joint joint3
- added joint joint1_base_rotation: type revolute, parent base, child base_link, origin xyz=0 0 0.110000 rpy=0 0 0, axis 0 0 1, limit lower=-3.14159265359 upper=3.14159265359 effort=1.0 velocity=2.0
- added joint joint2_shoulder: type revolute, parent base_link, child linker, origin xyz=0.00011040219 0.04143331674 0.04768605725 rpy=0 0 0, axis 0.976698944 0.214614011 0, limit lower=-3.14159265359 upper=3.14159265359 effort=1.0 velocity=2.0
- added joint joint3_wrist: type revolute, parent linker, child gripper, origin xyz=0.02489326226 -0.11328814381 0.03075909567 rpy=0 0 0, axis -0.976698944 -0.214614011 0, limit lower=-3.14159265359 upper=3.14159265359 effort=1.0 velocity=2.0
